Commit message: feat: simulation move to Gazebo (look logbook.txt for reason)

File: src/alfan_moveit_config/config/alfan_2025.ros2_control.xacro (robot description, xacro)
@@ -2,218 +2,309 @@
 <robot xmlns:xacro="http://www.ros.org/wiki/xacro">
     <xacro:macro name="alfan_2025_ros2_control" params="name initial_positions_file">
-        <xacro:property name="initial_positions" value="${load_yaml(initial_positions_file)['initial_positions']}"/>
+        <xacro:property name="initial_positions" value="${xacro.load_yaml(initial_positions_file)['initial_positions']}"/>
         <ros2_control name="${name}" type="system">
             <hardware>
                 <!-- By default, set up controllers for simulation. This won't work on real hardware -->
-                <plugin>mock_components/GenericSystem</plugin>
+                <plugin>ign_ros2_control/IgnitionSystem</plugin>
             </hardware>
             <joint name="head_yaw">
                 <command_interface name="position"/>
-                <command_interface name="velocity"/>
+                <!-- <command_interface name="velocity"/> -->
                 <state_interface name="position">
                   <param name="initial_value">${initial_positions['head_yaw']}</param>
                 </state_interface>
-                <state_interface name="velocity"/>
+                <!-- <state_interface name="velocity"/> -->
+                <param name="p">20.0</param>
+                <param name="d">0.5</param>
+                <param name="max_effort">2.5</param>
             </joint>
             <joint name="head_roll">
                 <command_interface name="position"/>
-                <command_interface name="velocity"/>
+                <!-- <command_interface name="velocity"/> -->
                 <state_interface name="position">
                   <param name="initial_value">${initial_positions['head_roll']}</param>
                 </state_interface>
-                <state_interface name="velocity"/>
+                <!-- <state_interface name="velocity"/> -->
+                <param name="p">20.0</param>
+                <param name="d">0.5</param>
+                <param name="max_effort">2.5</param>
             </joint>
             <joint name="r_hand_21">
                 <command_interface name="position"/>
-                <command_interface name="velocity"/>
+                <!-- <command_interface name="velocity"/> -->
                 <state_interface name="position">
                   <param name="initial_value">${initial_positions['r_hand_21']}</param>
                 </state_interface>
-                <state_interface name="velocity"/>
+                <!-- <state_interface name="velocity"/> -->
+                <param name="p">20.0</param>
+                <param name="d">0.5</param>
+                <param name="max_effort">2.5</param>
             </joint>
             <joint name="r_hand_22">
                 <command_interface name="position"/>
-                <command_interface name="velocity"/>
+                <!-- <command_interface name="velocity"/> -->
                 <state_interface name="position">
                   <param name="initial_value">${initial_positions['r_hand_22']}</param>
                 </state_interface>
-                <state_interface name="velocity"/>
+                <!-- <state_interface name="velocity"/> -->
+                <param name="p">20.0</param>
+                <param name="d">0.5</param>
+                <param name="max_effort">2.5</param>
             </joint>
             <joint name="r_hand_23">
                 <command_interface name="position"/>
-                <command_interface name="velocity"/>
+                <!-- <command_interface name="velocity"/> -->
                 <state_interface name="position">
                   <param name="initial_value">${initial_positions['r_hand_23']}</param>
                 </state_interface>
-                <state_interface name="velocity"/>
+                <!-- <state_interface name="velocity"/> -->
+                <param name="p">20.0</param>
+                <param name="d">0.5</param>
+                <param name="max_effort">2.5</param>
             </joint>
             <joint name="r_hand_24">
                 <command_interface name="position"/>
-                <command_interface name="velocity"/>
+                <!-- <command_interface name="velocity"/> -->
                 <state_interface name="position">
                   <param name="initial_value">${initial_positions['r_hand_24']}</param>
                 </state_interface>
-                <state_interface name="velocity"/>
+                <!-- <state_interface name="velocity"/> -->
+                <param name="p">20.0</param>
+                <param name="d">0.5</param>
+                <param name="max_effort">2.5</param>
             </joint>
             <joint name="r_hand_25">
                 <command_interface name="position"/>
-                <command_interface name="velocity"/>
+                <!-- <command_interface name="velocity"/> -->
                 <state_interface name="position">
                   <param name="initial_value">${initial_positions['r_hand_25']}</param>
                 </state_interface>
-                <state_interface name="velocity"/>
+                <!-- <state_interface name="velocity"/> -->
+                <param name="p">20.0</param>
+                <param name="d">0.5</param>
+                <param name="max_effort">2.5</param>
             </joint>
             <joint name="r_hand_26">
                 <command_interface name="position"/>
-                <command_interface name="velocity"/>
+                <!-- <command_interface name="velocity"/> -->
                 <state_interface name="position">
                   <param name="initial_value">${initial_positions['r_hand_26']}</param>
                 </state_interface>
-                <state_interface name="velocity"/>
+                <!-- <state_interface name="velocity"/> -->
+                <param name="p">20.0</param>
+                <param name="d">0.5</param>
+                <param name="max_effort">2.5</param>
             </joint>
             <joint name="l_hand_31">
                 <command_interface name="position"/>
-                <command_interface name="velocity"/>
+                <!-- <command_interface name="velocity"/> -->
                 <state_interface name="position">
                   <param name="initial_value">${initial_positions['l_hand_31']}</param>
                 </state_interface>
-                <state_interface name="velocity"/>
+                <!-- <state_interface name="velocity"/> -->
+                <param name="p">20.0</param>
+                <param name="d">0.5</param>
+                <param name="max_effort">2.5</param>
             </joint>
             <joint name="l_hand_32">
                 <command_interface name="position"/>
-                <command_interface name="velocity"/>
+                <!-- <command_interface name="velocity"/> -->
                 <state_interface name="position">
                   <param name="initial_value">${initial_positions['l_hand_32']}</param>
                 </state_interface>
-                <state_interface name="velocity"/>
+                <!-- <state_interface name="velocity"/> -->
+                <param name="p">20.0</param>
+                <param name="d">0.5</param>
+                <param name="max_effort">2.5</param>
             </joint>
             <joint name="l_hand_33">
                 <command_interface name="position"/>
-                <command_interface name="velocity"/>
+                <!-- <command_interface name="velocity"/> -->
                 <state_interface name="position">
                   <param name="initial_value">${initial_positions['l_hand_33']}</param>
                 </state_interface>
-                <state_interface name="velocity"/>
+                <!-- <state_interface name="velocity"/> -->
+                <param name="p">20.0</param>
+                <param name="d">0.5</param>
+                <param name="max_effort">2.5</param>
             </joint>
             <joint name="l_hand_34">
                 <command_interface name="position"/>
-                <command_interface name="velocity"/>
+                <!-- <command_interface name="velocity"/> -->
                 <state_interface name="position">
                   <param name="initial_value">${initial_positions['l_hand_34']}</param>
                 </state_interface>
-                <state_interface name="velocity"/>
+                <!-- <state_interface name="velocity"/> -->
+                <param name="p">20.0</param>
+                <param name="d">0.5</param>
+                <param name="max_effort">2.5</param>
             </joint>
             <joint name="l_hand_35">
                 <command_interface name="position"/>
-                <command_interface name="velocity"/>
+                <!-- <command_interface name="velocity"/> -->
                 <state_interface name="position">
                   <param name="initial_value">${initial_positions['l_hand_35']}</param>
                 </state_interface>
-                <state_interface name="velocity"/>
+                <!-- <state_interface name="velocity"/> -->
+                <param name="p">20.0</param>
+                <param name="d">0.5</param>
+                <param name="max_effort">2.5</param>
             </joint>
             <joint name="l_hand_36">
                 <command_interface name="position"/>
-                <command_interface name="velocity"/>
+                <!-- <command_interface name="velocity"/> -->
                 <state_interface name="position">
                   <param name="initial_value">${initial_positions['l_hand_36']}</param>
                 </state_interface>
-                <state_interface name="velocity"/>
+                <!-- <state_interface name="velocity"/> -->
+                <param name="p">20.0</param>
+                <param name="d">0.5</param>
+                <param name="max_effort">2.5</param>
             </joint>
             <joint name="r_hip_yaw">
                 <command_interface name="position"/>
-                <command_interface name="velocity"/>
+                <!-- <command_interface name="velocity"/> -->
                 <state_interface name="position">
                   <param name="initial_value">${initial_positions['r_hip_yaw']}</param>
                 </state_interface>
-                <state_interface name="velocity"/>
+                <!-- <state_interface name="velocity"/> -->
+                <param name="p">20.0</param>
+                <param name="d">0.5</param>
+                <param name="max_effort">2.5</param>
             </joint>
             <joint name="r_hip_roll">
                 <command_interface name="position"/>
-                <command_interface name="velocity"/>
+                <!-- <command_interface name="velocity"/> -->
                 <state_interface name="position">
                   <param name="initial_value">${initial_positions['r_hip_roll']}</param>
                 </state_interface>
-                <state_interface name="velocity"/>
+                <!-- <state_interface name="velocity"/> -->
+                <param name="p">20.0</param>
+                <param name="d">0.5</param>
+                <param name="max_effort">2.5</param>
             </joint>
             <joint name="r_hip_pitch">
                 <command_interface name="position"/>
-                <command_interface name="velocity"/>
+                <!-- <command_interface name="velocity"/> -->
                 <state_interface name="position">
                   <param name="initial_value">${initial_positions['r_hip_pitch']}</param>
                 </state_interface>
-                <state_interface name="velocity"/>
+                <!-- <state_interface name="velocity"/> -->
+                <param name="p">20.0</param>
+                <param name="d">0.5</param>
+                <param name="max_effort">2.5</param>
             </joint>
             <joint name="r_knee">
                 <command_interface name="position"/>
-                <command_interface name="velocity"/>
+                <!-- <command_interface name="velocity"/> -->
                 <state_interface name="position">
                   <param name="initial_value">${initial_positions['r_knee']}</param>
                 </state_interface>
-                <state_interface name="velocity"/>
+                <!-- <state_interface name="velocity"/> -->
+                <param name="p">20.0</param>
+                <param name="d">0.5</param>
+                <param name="max_effort">2.5</param>
             </joint>
             <joint name="r_ankle_pitch">
                 <command_interface name="position"/>
-                <command_interface name="velocity"/>
+                <!-- <command_interface name="velocity"/> -->
                 <state_interface name="position">
                   <param name="initial_value">${initial_positions['r_ankle_pitch']}</param>
                 </state_interface>
-                <state_interface name="velocity"/>
+                <!-- <state_interface name="velocity"/> -->
+                <param name="p">20.0</param>
+                <param name="d">0.5</param>
+                <param name="max_effort">2.5</param>
             </joint>
             <joint name="r_ankle_roll">
                 <command_interface name="position"/>
-                <command_interface name="velocity"/>
+                <!-- <command_interface name="velocity"/> -->
                 <state_interface name="position">
                   <param name="initial_value">${initial_positions['r_ankle_roll']}</param>
                 </state_interface>
-                <state_interface name="velocity"/>
+                <!-- <state_interface name="velocity"/> -->
+                <param name="p">20.0</param>
+                <param name="d">0.5</param>
+                <param name="max_effort">2.5</param>
             </joint>
             <joint name="l_hip_yaw">
                 <command_interface name="position"/>
-                <command_interface name="velocity"/>
+                <!-- <command_interface name="velocity"/> -->
                 <state_interface name="position">
                   <param name="initial_value">${initial_positions['l_hip_yaw']}</param>
                 </state_interface>
-                <state_interface name="velocity"/>
+                <!-- <state_interface name="velocity"/> -->
+                <param name="p">20.0</param>
+                <param name="d">0.5</param>
+                <param name="max_effort">2.5</param>
             </joint>
             <joint name="l_hip_roll">
                 <command_interface name="position"/>
-                <command_interface name="velocity"/>
+                <!-- <command_interface name="velocity"/> -->
                 <state_interface name="position">
                   <param name="initial_value">${initial_positions['l_hip_roll']}</param>
                 </state_interface>
-                <state_interface name="velocity"/>
+                <!-- <state_interface name="velocity"/> -->
+                <param name="p">20.0</param>
+                <param name="d">0.5</param>
+                <param name="max_effort">2.5</param>
             </joint>
             <joint name="l_hip_pitch">
                 <command_interface name="position"/>
-                <command_interface name="velocity"/>
+                <!-- <command_interface name="velocity"/> -->
                 <state_interface name="position">
                   <param name="initial_value">${initial_positions['l_hip_pitch']}</param>
                 </state_interface>
-                <state_interface name="velocity"/>
+                <!-- <state_interface name="velocity"/> -->
+                <param name="p">20.0</param>
+                <param name="d">0.5</param>
+                <param name="max_effort">2.5</param>
             </joint>
             <joint name="l_knee">
                 <command_interface name="position"/>
-                <command_interface name="velocity"/>
+                <!-- <command_interface name="velocity"/> -->
                 <state_interface name="position">
                   <param name="initial_value">${initial_positions['l_knee']}</param>
                 </state_interface>
-                <state_interface name="velocity"/>
+                <!-- <state_interface name="velocity"/> -->
+                <param name="p">20.0</param>
+                <param name="d">0.5</param>
+                <param name="max_effort">2.5</param>
             </joint>
             <joint name="l_ankle_pitch">
                 <command_interface name="position"/>
-                <command_interface name="velocity"/>
+                <!-- <command_interface name="velocity"/> -->
                 <state_interface name="position">
                   <param name="initial_value">${initial_positions['l_ankle_pitch']}</param>
                 </state_interface>
-                <state_interface name="velocity"/>
+                <!-- <state_interface name="velocity"/> -->
+                <param name="p">20.0</param>
+                <param name="d">0.5</param>
+                <param name="max_effort">2.5</param>
             </joint>
             <joint name="l_ankle_roll">
                 <command_interface name="position"/>
-                <command_interface name="velocity"/>
+                <!-- <command_interface name="velocity"/> -->
                 <state_interface name="position">
                   <param name="initial_value">${initial_positions['l_ankle_roll']}</param>
                 </state_interface>
-                <state_interface name="velocity"/>
-            </joint>
+                <!-- <state_interface name="velocity"/> -->
+                <param name="p">20.0</param>
+                <param name="d">0.5</param>
+                <param name="max_effort">2.5</param>
+            </joint>
+            <!-- 6 Axis IMU Sensor -->
+            <sensor name="imu_sensor">
+              <state_interface name="orientation.x"/>
+              <state_interface name="orientation.y"/>
+              <state_interface name="orientation.z"/>
+              <state_interface name="orientation.w"/>
+              <state_interface name="angular_velocity.x"/>
+              <state_interface name="angular_velocity.y"/>
+              <state_interface name="angular_velocity.z"/>
+              <state_interface name="linear_acceleration.x"/>
+              <state_interface name="linear_acceleration.y"/>
+              <state_interface name="linear_acceleration.z"/>
+            </sensor>
         </ros2_control>
     </xacro:macro>

File: src/alfan_moveit_config/config/alfan_2025.urdf.xacro (robot description, xacro)
@@ -6,4 +6,9 @@
     <!-- Import control_xacro -->
     <xacro:include filename="alfan_2025.ros2_control.xacro" />
-    <xacro:alfan_2025_ros2_control name="FakeSystem" initial_positions_file="$(arg initial_positions_file)"/>
+    <xacro:alfan_2025_ros2_control name="GazeboROS2" initial_positions_file="$(arg initial_positions_file)"/>
+    <gazebo>
+        <plugin filename="ign_ros2_control-system" name="ign_ros2_control::IgnitionROS2ControlPlugin">
+            <parameters>$(find alfan_moveit_config)/config/ros2_controllers.yaml</parameters>
+        </plugin>
+    </gazebo>
 </robot>
