Commit message: feat: simulation move to Gazebo (look logbook.txt for reason)

File: src/alfan_robot_description/urdf/alfan.urdf (robot description, URDF)
Before this commit: robot alfan_2025, 28 links, 27 joints
Links:
- added link imu_link, mass 0.001
- link body: geometry collision box size=0.113618 0.0647698 0.097; collision box size=0.124589 0.0459933 0.113
- link head_to_face: geometry collision box size=0.032099 0.0505201 0.044; visual mesh filename=file://$(find alfan_robot_description)/meshes/head_to_face.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
- link hip_connector: geometry collision box size=0.0505652 0.0271414 0.0343; visual mesh filename=file://$(find alfan_robot_description)/meshes/hip_connector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
- link hip_connector_2: geometry collision box size=0.0505652 0.0271414 0.0343; visual mesh filename=file://$(find alfan_robot_description)/meshes/hip_connector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
- link l_ankle_mx28_block: geometry collision box size=0.0841545 0.043397 0.051; visual mesh filename=file://$(find alfan_robot_description)/meshes/l_ankle_mx28_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
- link l_arm_pitch: geometry collision box size=0.0286099 0.0240448 0.038; visual mesh filename=file://$(find alfan_robot_description)/meshes/l_arm_pitch.s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
- link l_elbow_block: geometry collision box size=0.0312457 0.0521967 0.039; visual mesh filename=file://$(find alfan_robot_description)/meshes/l_elbow_block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
- link l_foot: geometry collision box size=0.0271116 0.0438503 0.054; collision box size=0.119957 0.0800615 0.01
- link l_hip_mx28_block: geometry collision box size=0.0860053 0.0422632 0.051; visual mesh filename=file://$(find alfan_robot_description)/meshes/l_hip_mx28_bl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
- link l_hip_to_knee: geometry collision box size=0.0357598 0.0454412 0.108; visual mesh filename=file://$(find alfan_robot_description)/meshes/l_hip_to_knee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
- link l_palm: geometry collision box size=0.0373386 0.0354738 0.086; visual mesh filename=file://$(find alfan_robot_description)/meshes/l_palm.stl
- link l_shoulder_connector: geometry collision box size=0.038113 0.0359998 0.029; visual mesh filename=file://$(find alfan_robot_description)/meshes/l_shoulder_co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
- link l_wrist_pitch: geometry collision box size=0.0313319 0.0241859 0.038; visual mesh filename=file://$(find alfan_robot_description)/meshes/l_wrist_pitch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
- link l_wrist_roll: geometry collision box size=0.0340405 0.0500191 0.042; visual mesh filename=file://$(find alfan_robot_description)/meshes/l_wrist_roll.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
- link neck: geometry collision box size=0.0240336 0.039947 0.029; visual mesh filename=file://$(find alfan_robot_description)/meshes/neck.stl
- link r_ankle_mx28_block: geometry collision box size=0.0840214 0.0432827 0.051; visual mesh filename=file://$(find alfan_robot_description)/meshes/r_ankle_mx28_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
- link r_arm_pitch: geometry collision box size=0.0286122 0.0241427 0.038; visual mesh filename=file://$(find alfan_robot_description)/meshes/r_arm_pitch.s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
- link r_elbow_block: geometry collision box size=0.0311226 0.0520685 0.039; visual mesh filename=file://$(find alfan_robot_description)/meshes/r_elbow_block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
- link r_foot: geometry collision box size=0.0272329 0.0438661 0.054; collision box size=0.120686 0.080481 0.01
- link r_hip_mx28_block: geometry collision box size=0.086166 0.0433161 0.051; visual mesh filename=file://$(find alfan_robot_description)/meshes/r_hip_mx28_bl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
- link r_hip_to_knee: geometry collision box size=0.0357519 0.0454254 0.108; visual mesh filename=file://$(find alfan_robot_description)/meshes/r_hip_to_knee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
- link r_palm: geometry collision box size=0.0370488 0.0352658 0.086; visual mesh filename=file://$(find alfan_robot_description)/meshes/r_palm.stl
- link r_shoulder_connector: geometry collision box size=0.0381521 0.0360597 0.029; visual mesh filename=file://$(find alfan_robot_description)/meshes/r_shoulder_co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
- link r_wrist_pitch: geometry collision box size=0.0313399 0.0243173 0.038; visual mesh filename=file://$(find alfan_robot_description)/meshes/r_wrist_pitch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
- link r_wrist_roll: geometry collision box size=0.0341979 0.050073 0.042; visual mesh filename=file://$(find alfan_robot_description)/meshes/r_wrist_roll.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
- link tibia: geometry collision box size=0.105526 0.0398408 0.045; visual mesh filename=file://$(find alfan_robot_description)/meshes/tibia.stl
- link tibia_2: geometry collision box size=0.105526 0.0398408 0.045; visual mesh filename=file://$(find alfan_robot_description)/meshes/tibia.stl
Joints:
- added joint imu_joint: type fixed, parent body, child imu_link, origin xyz=0.0 0.0 -0.0580833 rpy=0 0 1.5708
- joint base_to_body: origin (none) -> xyz=0 0 0 rpy=0 0 1.5708
- joint head_roll: limit lower=-3.141592653589793 upper=3.141592653589793 effort=10.0 velocity=10.0 -> lower=-3.141592653589793 upper=3.141592653589793 effort=2.5 velocity=10.0
- joint head_yaw: limit lower=-3.141592653589793 upper=3.141592653589793 effort=10.0 velocity=10.0 -> lower=-3.141592653589793 upper=3.141592653589793 effort=2.5 velocity=10.0
- joint l_ankle_pitch: limit lower=-3.14159 upper=3.14159 effort=10.0 velocity=10.0 -> lower=-1.5708 upper=1.5708 effort=2.5 velocity=10.0
- joint l_ankle_roll: limit lower=-3.14159 upper=3.14159 effort=10.0 velocity=10.0 -> lower=-0.3491 upper=0.3491 effort=2.5 velocity=10.0
- joint l_hand_31: limit lower=-3.49066 upper=1.5708 effort=10.0 velocity=10.0 -> lower=-3.49066 upper=1.5708 effort=2.5 velocity=10.0
- joint l_hand_32: limit lower=-1.8326 upper=3.40339 effort=10.0 velocity=10.0 -> lower=-1.8326 upper=3.40339 effort=2.5 velocity=10.0
- joint l_hand_33: limit lower=-3.14159 upper=2.0944 effort=10.0 velocity=10.0 -> lower=-3.14159 upper=2.0944 effort=2.5 velocity=10.0
- joint l_hand_34: limit lower=0 upper=1.74533 effort=10.0 velocity=10.0 -> lower=0 upper=1.74533 effort=2.5 velocity=10.0
- joint l_hand_35: limit lower=-1.8326 upper=3.40339 effort=10.0 velocity=10.0 -> lower=-1.8326 upper=3.40339 effort=2.5 velocity=10.0
- joint l_hand_36: limit lower=-1.74533 upper=1.74533 effort=10.0 velocity=10.0 -> lower=-1.74533 upper=1.74533 effort=2.5 velocity=10.0
- joint l_hip_pitch: limit lower=-3.14159 upper=3.14159 effort=10.0 velocity=10.0 -> lower=-0.5235987756 upper=1.5707963268 effort=2.5 velocity=10.0
- joint l_hip_roll: limit lower=-3.14159 upper=3.14159 effort=10.0 velocity=10.0 -> lower=-0.78538982 upper=0.78538982 effort=2.5 velocity=10.0
- joint l_hip_yaw: limit lower=-3.14159 upper=3.14159 effort=10.0 velocity=10.0 -> lower=-0.43633 upper=0.43633 effort=2.5 velocity=10.0
- joint l_knee: limit lower=-3.14159 upper=3.14159 effort=10.0 velocity=10.0 -> lower=-3.14159 upper=0.0 effort=2.5 velocity=10.0
- joint r_ankle_pitch: limit lower=-3.14159 upper=3.14159 effort=10.0 velocity=10.0 -> lower=-1.5708 upper=1.5708 effort=2.5 velocity=10.0
- joint r_ankle_roll: limit lower=-3.14159 upper=3.14159 effort=10.0 velocity=10.0 -> lower=-0.3491 upper=0.3491 effort=2.5 velocity=10.0
- joint r_hand_21: limit lower=-1.57078 upper=3.49067 effort=10.0 velocity=10.0 -> lower=-1.57078 upper=3.49067 effort=2.5 velocity=10.0
- joint r_hand_22: limit lower=-3.40339 upper=1.8326 effort=10.0 velocity=10.0 -> lower=-3.40339 upper=1.8326 effort=2.5 velocity=10.0
- joint r_hand_23: limit lower=-2.09439 upper=3.1416 effort=10.0 velocity=10.0 -> lower=-2.09439 upper=3.1416 effort=2.5 velocity=10.0
- joint r_hand_24: limit lower=-1.74533 upper=4.19964e-06 effort=10.0 velocity=10.0 -> lower=-1.74533 upper=4.19964e-06 effort=2.5 velocity=10.0
- joint r_hand_25: limit lower=-3.40339 upper=1.8326 effort=10.0 velocity=10.0 -> lower=-3.40339 upper=1.8326 effort=2.5 velocity=10.0
- joint r_hand_26: limit lower=-1.74532 upper=1.74534 effort=10.0 velocity=10.0 -> lower=-1.74532 upper=1.74534 effort=2.5 velocity=10.0
- joint r_hip_pitch: limit lower=-3.14159 upper=3.14159 effort=10.0 velocity=10.0 -> lower=-1.5707963268 upper=0.5235987756 effort=2.5 velocity=10.0
- joint r_hip_roll: limit lower=-3.14159 upper=3.14159 effort=10.0 velocity=10.0 -> lower=-0.78538982 upper=0.78538982 effort=2.5 velocity=10.0
- joint r_hip_yaw: limit lower=-3.14159 upper=3.14159 effort=10.0 velocity=10.0 -> lower=-0.43633 upper=0.43633 effort=2.5 velocity=10.0
- joint r_knee: limit lower=-3.14159 upper=3.14159 effort=10.0 velocity=10.0 -> lower=0.0 upper=3.14159 effort=2.5 velocity=10.0
