Commit message: fix: simulation and URDF

File: src/alfan_robot_description/urdf/alfan.urdf (robot description, URDF)
Before this commit: robot alfan_2025, 29 links, 28 joints
Links:
- link body: mass 0.776 -> 0.757108; geometry collision box size=0.0648476 0.123854 0.097; collision box size=0.124687 0.0458965 0.113
- link head_to_face: mass 0.043 -> 0.035939
- link hip_connector: mass 0.0123061 -> 0.0123973; geometry collision box size=0.0506482 0.0270708 0.035; visual mesh filename=file://$(find alfan_robot_description)/meshes/hip_connector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
- link hip_connector_2: mass 0.0123061 -> 0.0123973; geometry collision box size=0.0506482 0.0270708 0.035; visual mesh filename=file://$(find alfan_robot_description)/meshes/hip_connector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
- link l_ankle_mx28_block: mass 0.171 -> 0.162255; geometry collision box size=0.0840214 0.0432827 0.051; visual mesh filename=file://$(find alfan_robot_description)/meshes/l_ankle_mx28_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
- link l_arm_pitch: mass 0.021 -> 0.020676; geometry collision box size=0.0286122 0.0240341 0.038; visual mesh filename=file://$(find alfan_robot_description)/meshes/l_arm_pitch.s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
- link l_elbow_block: mass 0.041 -> 0.040594; geometry collision box size=0.0312596 0.0520685 0.039; visual mesh filename=file://$(find alfan_robot_description)/meshes/l_elbow_block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
- link l_foot: mass 0.068074 -> 0.063842; geometry collision box size=0.0221666 0.0438909 0.054; collision box size=0.120001 0.0800676 0.003
- link l_hip_mx28_block: mass 0.172 -> 0.162255; geometry collision box size=0.0859449 0.0423941 0.051; visual mesh filename=file://$(find alfan_robot_description)/meshes/l_hip_mx28_bl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
- link l_hip_to_knee: mass 0.1 -> 0.095285; geometry collision box size=0.03584 0.0455282 0.108; visual mesh filename=file://$(find alfan_robot_description)/meshes/l_hip_to_knee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
- link l_palm: mass 0.027 -> 0.024199; geometry collision box size=0.0374329 0.0262008 0.086; visual mesh filename=file://$(find alfan_robot_description)/meshes/l_palm.stl
- link l_shoulder_connector: geometry collision box size=0.0290724 0.0380736 0.036; visual mesh filename=file://$(find alfan_robot_description)/meshes/l_shoulder_co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
- link l_wrist_pitch: mass 0.021 -> 0.020676; geometry collision box size=0.0312241 0.0240341 0.038; visual mesh filename=file://$(find alfan_robot_description)/meshes/l_wrist_pitch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
- link l_wrist_roll: mass 0.024 -> 0.023692; geometry collision box size=0.0340473 0.0499962 0.042; visual mesh filename=file://$(find alfan_robot_description)/meshes/l_wrist_roll.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
- link neck: mass 0.025 -> 0.029997; geometry collision box size=0.0240336 0.039947 0.031; visual mesh filename=file://$(find alfan_robot_description)/meshes/neck.stl
- link r_ankle_mx28_block: mass 0.171 -> 0.162255
- link r_arm_pitch: mass 0.021 -> 0.020676; geometry collision box size=0.0286122 0.0240341 0.038; visual mesh filename=file://$(find alfan_robot_description)/meshes/r_arm_pitch.s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
- link r_elbow_block: mass 0.041 -> 0.040594
- link r_foot: mass 0.068074 -> 0.063842; geometry collision box size=0.0221666 0.0438909 0.054; collision box size=0.120001 0.0800676 0.003
- link r_hip_mx28_block: mass 0.172 -> 0.162255
- link r_hip_to_knee: mass 0.1 -> 0.095285; geometry collision box size=0.03584 0.0455282 0.108; visual mesh filename=file://$(find alfan_robot_description)/meshes/r_hip_to_knee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
- link r_palm: mass 0.027 -> 0.024199; geometry collision box size=0.0370488 0.0262008 0.086; visual mesh filename=file://$(find alfan_robot_description)/meshes/r_palm.stl
- link r_shoulder_connector: geometry collision box size=0.0290761 0.0380915 0.036; visual mesh filename=file://$(find alfan_robot_description)/meshes/r_shoulder_co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
- link r_wrist_pitch: mass 0.021 -> 0.020676; geometry collision box size=0.0312241 0.0240341 0.038; visual mesh filename=file://$(find alfan_robot_description)/meshes/r_wrist_pitch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
- link r_wrist_roll: mass 0.024 -> 0.023692; geometry collision box size=0.0340473 0.0501498 0.042; visual mesh filename=file://$(find alfan_robot_description)/meshes/r_wrist_roll.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
- link tibia: mass 0.0331521 -> 0.0333977; geometry collision box size=0.039678 0.105746 0.045; visual mesh filename=file://$(find alfan_robot_description)/meshes/tibia.stl
- link tibia_2: mass 0.0331521 -> 0.0333977; geometry collision box size=0.039678 0.105746 0.045; visual mesh filename=file://$(find alfan_robot_description)/meshes/tibia.stl
Joints:
- removed joint base_to_body
- added joint base_link_to_body: type fixed, parent base_link, child body, origin xyz=0 0 0 rpy=0 0 0
- joint head_roll: limit lower=-3.141592653589793 upper=3.141592653589793 effort=2.5 velocity=10.0 -> lower=-0.785398 upper=0.785398 effort=10 velocity=10; origin xyz=-0.015 -2.87625e-09 0.03092 rpy=1.5708 3.20936e-15 -1.5708 -> xyz=0.015 -1.15463e-16 0.03092 rpy=1.5708 -0 1.5708
- joint head_yaw: limit lower=-3.141592653589793 upper=3.141592653589793 effort=2.5 velocity=10.0 -> lower=-0.523599 upper=0.523599 effort=10 velocity=10; origin xyz=8.10306e-05 0.0362866 0.390889 rpy=1.9557e-09 -0.0104304 1.5708 -> xyz=-0.011357 3.60385e-08 0.392755 rpy=-3.07442e-13 1.17186e-15 -2.77556e-17
- joint l_ankle_pitch: limit lower=-1.5708 upper=1.5708 effort=2.5 velocity=10.0 -> lower=-1.5708 upper=1.22173 effort=10 velocity=10; origin xyz=0.093 3.46945e-18 -3.46945e-18 rpy=1.53445e-24 -6.12517e-17 -1.5708 -> xyz=-0.093 4.21538e-16 1.04083e-17 rpy=2.06189e-29 -1.51461e-28 5.55112e-17; parent tibia_2 -> tibia
- joint l_ankle_roll: limit lower=-0.3491 upper=0.3491 effort=2.5 velocity=10.0 -> lower=-0.375246 upper=0.375246 effort=10 velocity=10; origin xyz=0.02305 -3.39034e-14 -0.01995 rpy=-3.14159 1.5708 0 -> xyz=3.07393e-14 -0.02305 0.01995 rpy=-1.5708 -1.5708 0
- joint l_hand_31: limit lower=-3.49066 upper=1.5708 effort=2.5 velocity=10.0 -> lower=-3.14159 upper=3.14159 effort=10 velocity=10; origin xyz=0.0589788 0.0152645 0.365421 rpy=-1.87514e-07 1.5708 0 -> xyz=0.00996904 0.058983 0.367555 rpy=-1.5708 -1.5708 0
- joint l_hand_32: limit lower=-1.8326 upper=3.40339 effort=2.5 velocity=10.0 -> lower=-2.61799 upper=1.5708 effort=10 velocity=10; origin xyz=0.016 -0.01595 0.018 rpy=1.5708 -0.776672 -2.06163e-16 -> xyz=-0.016 0.01595 0.018 rpy=-1.5708 -1.5708 0
- joint l_hand_33: limit lower=-3.14159 upper=2.0944 effort=2.5 velocity=10.0 -> lower=-3.14159 upper=3.14159 effort=10 velocity=10; origin xyz=0.029 -4.38538e-15 -0.0145 rpy=-1.5708 -3.77924e-13 1.5708 -> xyz=0.029 -5.67324e-14 -0.0145 rpy=1.5708 3.4138e-28 1.5708
- joint l_hand_34: limit lower=0 upper=1.74533 effort=2.5 velocity=10.0 -> lower=0 upper=2.0944 effort=10 velocity=10; origin xyz=-0.0144 -7.69003e-15 -0.04 rpy=-3.28224e-13 1.5708 0 -> xyz=3.10862e-15 0.0144 0.04 rpy=-1.5708 -1.5708 0
- joint l_hand_35: limit lower=-1.8326 upper=3.40339 effort=2.5 velocity=10.0 -> lower=-3.14159 upper=3.14159 effort=10 velocity=10; origin xyz=0.0386011 -0.00300003 0.01695 rpy=3.14159 -1.5708 0 -> xyz=0.0409 0.003 -0.01545 rpy=1.5708 -6.82466e-16 1.5708
- joint l_hand_36: limit lower=-1.74533 upper=1.74533 effort=2.5 velocity=10.0 -> lower=-1.7017 upper=1.7017 effort=10 velocity=10; origin xyz=-0.0154 -9.61037e-16 0.029 rpy=1.13408e-16 -1.5708 0 -> xyz=-9.4369e-16 0.0154 0.029 rpy=-1.5708 -1.5708 0
- joint l_hip_pitch: limit lower=-0.5235987756 upper=1.5707963268 effort=2.5 velocity=10.0 -> lower=-2.35619 upper=0.497419 effort=10 velocity=10; origin xyz=-0.01995 -3.19242e-10 0.02305 rpy=3.14159 1.5708 0 -> xyz=-0.01995 -6.07486e-13 0.02305 rpy=1.5708 6.4443e-19 1.5708
- joint l_hip_roll: limit lower=-0.78538982 upper=0.78538982 effort=2.5 velocity=10.0 -> lower=-0.375246 upper=0.375246 effort=10 velocity=10; origin xyz=-0.028 1.52656e-16 0.0317982 rpy=-1.5708 -2.9301e-15 -1.5708 -> xyz=-0.028 0 -0.0317982 rpy=1.5708 -0 1.5708; parent hip_connector_2 -> hip_connector
- joint l_hip_yaw: child hip_connector_2 -> hip_connector; limit lower=-0.43633 upper=0.43633 effort=2.5 velocity=10.0 -> lower=-0.523599 upper=0.523599 effort=10 velocity=10; origin xyz=0.0444 0.0225 0.250434 rpy=3.14159 2.23241e-25 -1.5708 -> xyz=0.00275 0.0444 0.252434 rpy=-3.07436e-13 1.17478e-15 -1.33488e-16
- joint l_knee: child tibia_2 -> tibia; limit lower=-3.14159 upper=0.0 effort=2.5 velocity=10.0 -> lower=0 upper=2.61799 effort=10 velocity=10; origin xyz=6.32584e-13 0.0938373 -0.000550036 rpy=7.6929e-14 1.35379e-14 1.5708 -> xyz=-0.0938373 -2.02966e-12 0.000550036 rpy=1.01253e-24 -1.62064e-26 5.55112e-17
- joint r_ankle_pitch: limit lower=-1.5708 upper=1.5708 effort=2.5 velocity=10.0 -> lower=-1.5708 upper=1.22173 effort=10 velocity=10; origin xyz=0.093 0 1.38778e-17 rpy=-2.22045e-16 -6.13031e-17 1.5708 -> xyz=-0.093 -3.90313e-18 -3.46945e-18 rpy=1.55505e-36 -0 6.88016e-28; parent tibia -> tibia_2
- joint r_ankle_roll: limit lower=-0.3491 upper=0.3491 effort=2.5 velocity=10.0 -> lower=-0.375246 upper=0.375246 effort=10 velocity=10; origin xyz=0.02305 -2.60209e-15 -0.01995 rpy=-7.45549e-13 -1.5708 0 -> xyz=6.0292e-14 -0.02305 -0.01995 rpy=-1.5708 -1.5708 0
- joint r_hand_21: limit lower=-1.57078 upper=3.49067 effort=2.5 velocity=10.0 -> lower=-3.14159 upper=3.14159 effort=10 velocity=10; origin xyz=-0.058987 0.0152644 0.365421 rpy=-1.5708 1.57078 1.5708 -> xyz=0.00996904 -0.0589829 0.367555 rpy=-1.5708 -1.5708 0
- joint r_hand_22: limit lower=-3.40339 upper=1.8326 effort=2.5 velocity=10.0 -> lower=-1.5708 upper=2.61799 effort=10 velocity=10; origin xyz=0.016 0.01595 0.018 rpy=-1.5708 0.776672 -9.454e-15 -> xyz=-0.016 0.01595 -0.018 rpy=-1.5708 -1.5708 0
- joint r_hand_23: limit lower=-2.09439 upper=3.1416 effort=2.5 velocity=10.0 -> lower=-3.14159 upper=3.14159 effort=10 velocity=10; origin xyz=3.38618e-15 -0.029 -0.0145 rpy=1.5708 8.47445e-06 -3.14159 -> xyz=-0.029 -8.38218e-15 -0.0145 rpy=1.5708 -0 1.5708
- joint r_hand_24: limit lower=-1.74533 upper=4.19964e-06 effort=2.5 velocity=10.0 -> lower=-2.0944 upper=0 effort=10 velocity=10; origin xyz=-0.0144 7.71258e-15 -0.04 rpy=-1.5708 1.57079 1.5708 -> xyz=1.2379e-14 0.0144 -0.04 rpy=-1.5708 -1.5708 0
- joint r_hand_25: limit lower=-3.40339 upper=1.8326 effort=2.5 velocity=10.0 -> lower=-3.14159 upper=3.14159 effort=10 velocity=10; origin xyz=0.041 -0.003 -0.01545 rpy=-5.86012e-22 1.5708 0 -> xyz=-0.041 0.003 -0.01545 rpy=1.5708 -0 1.5708
- joint r_hand_26: limit lower=-1.74532 upper=1.74534 effort=2.5 velocity=10.0 -> lower=-1.7017 upper=1.7017 effort=10 velocity=10; origin xyz=-0.0154 1.05818e-15 0.029 rpy=1.5708 -1.57079 -1.5708 -> xyz=-7.21645e-16 0.0154 -0.029 rpy=-1.5708 -1.5708 0
- joint r_hip_pitch: limit lower=-1.5707963268 upper=0.5235987756 effort=2.5 velocity=10.0 -> lower=-2.35619 upper=0.497419 effort=10 velocity=10; origin xyz=0.01995 -4.28185e-13 0.02305 rpy=2.15155e-11 1.5708 0 -> xyz=0.01995 1.33227e-15 0.02305 rpy=1.5708 -6.88016e-28 1.5708
- joint r_hip_roll: limit lower=-0.78538982 upper=0.78538982 effort=2.5 velocity=10.0 -> lower=-0.375246 upper=0.375246 effort=10 velocity=10; origin xyz=-0.028 -2.77556e-17 0.0317982 rpy=-1.5708 3.58391e-14 -1.5708 -> xyz=-0.028 -6.93889e-18 -0.0317982 rpy=1.5708 -0 1.5708; parent hip_connector -> hip_connector_2
- joint r_hip_yaw: child hip_connector -> hip_connector_2; limit lower=-0.43633 upper=0.43633 effort=2.5 velocity=10.0 -> lower=-0.523599 upper=0.523599 effort=10 velocity=10; origin xyz=-0.0444 0.0225 0.250434 rpy=3.14159 -2.83277e-16 -1.5708 -> xyz=0.00275 -0.0444 0.252434 rpy=-3.07442e-13 1.51693e-23 -2.77556e-17
- joint r_knee: child tibia -> tibia_2; limit lower=0.0 upper=3.14159 effort=2.5 velocity=10.0 -> lower=0 upper=2.61799 effort=10 velocity=10; origin xyz=2.70121e-13 -0.0938373 -0.000550036 rpy=2.24345e-20 2.22045e-16 -1.5708 -> xyz=-0.0938373 3.16515e-13 -0.000550036 rpy=1.55484e-36 -0 6.88002e-28
